Commit message: make default URDF

File: public/default.urdf (robot description, URDF)
Before this commit: robot five_finger_hand, 16 links, 15 joints
Links:
- added link thumb_mount; visual box size=0.001 0.001 0.001
Joints:
- added joint thumb_abduction_joint: type revolute, parent base, child thumb_mount, origin xyz=-0.035 0 0.0 rpy=0 0 0, axis 0 0 1, limit lower=-0.5 upper=0.5 effort=1.0 velocity=1.0
- joint index_base_joint: axis 1 0 0 -> -1 0 0; limit lower=-0.2 upper=0.8 effort=1.0 velocity=1.0 -> lower=0.0 upper=1.6 effort=1.0 velocity=1.0
- joint index_mid_joint: axis 1 0 0 -> -1 0 0; limit lower=0.0 upper=1.5 effort=1.0 velocity=1.0 -> lower=0.0 upper=1.6 effort=1.0 velocity=1.0
- joint index_tip_joint: axis 1 0 0 -> -1 0 0; limit lower=0.0 upper=1.2 effort=1.0 velocity=1.0 -> lower=0.0 upper=1.6 effort=1.0 velocity=1.0
- joint middle_base_joint: axis 1 0 0 -> -1 0 0; limit lower=-0.2 upper=0.8 effort=1.0 velocity=1.0 -> lower=0.0 upper=1.6 effort=1.0 velocity=1.0
- joint middle_mid_joint: axis 1 0 0 -> -1 0 0; limit lower=0.0 upper=1.5 effort=1.0 velocity=1.0 -> lower=0.0 upper=1.6 effort=1.0 velocity=1.0
- joint middle_tip_joint: axis 1 0 0 -> -1 0 0; limit lower=0.0 upper=1.2 effort=1.0 velocity=1.0 -> lower=0.0 upper=1.6 effort=1.0 velocity=1.0
- joint pinky_base_joint: axis 1 0 0 -> -1 0 0; limit lower=-0.2 upper=0.8 effort=1.0 velocity=1.0 -> lower=0.0 upper=1.6 effort=1.0 velocity=1.0
- joint pinky_mid_joint: axis 1 0 0 -> -1 0 0; limit lower=0.0 upper=1.5 effort=1.0 velocity=1.0 -> lower=0.0 upper=1.6 effort=1.0 velocity=1.0
- joint pinky_tip_joint: axis 1 0 0 -> -1 0 0; limit lower=0.0 upper=1.2 effort=1.0 velocity=1.0 -> lower=0.0 upper=1.6 effort=1.0 velocity=1.0
- joint ring_base_joint: axis 1 0 0 -> -1 0 0; limit lower=-0.2 upper=0.8 effort=1.0 velocity=1.0 -> lower=0.0 upper=1.6 effort=1.0 velocity=1.0
- joint ring_mid_joint: axis 1 0 0 -> -1 0 0; limit lower=0.0 upper=1.5 effort=1.0 velocity=1.0 -> lower=0.0 upper=1.6 effort=1.0 velocity=1.0
- joint ring_tip_joint: axis 1 0 0 -> -1 0 0; limit lower=0.0 upper=1.2 effort=1.0 velocity=1.0 -> lower=0.0 upper=1.6 effort=1.0 velocity=1.0
- joint thumb_base_joint: origin xyz=-0.035 0 0.06 rpy=0 0 0 -> xyz=0 0 0 rpy=0 0 0; parent base -> thumb_mount
- joint thumb_mid_joint: origin xyz=0 0 0.03 rpy=0 0 0 -> xyz=0 0.03 0 rpy=0 0 0
- joint thumb_tip_joint: axis 0 1 0 -> 1 0 0; origin xyz=0 0 0.025 rpy=0 0 0 -> xyz=0 0.025 0 rpy=0 0 0

File: public/hand_4dof.urdf (robot description, URDF)
Before this commit: robot five_finger_hand_4dof, 21 links, 20 joints
Joints:
- joint thumb_roll_joint: origin xyz=0.04 0.025 0.02 rpy=0 0 3.14159 -> xyz=0.045 0.01 0.02 rpy=0 -0.785 -1.5708
